Commit message: feat(simulation): complete Stage 1 - MuJoCo digital twin, scene, virtual sensors, and tests

File: urdf_model/root_mujoco.urdf (robot description, URDF)
Before this commit: robot root, 8 links, 7 joints
Links:
- link 1_сустав__1__1__body1: geometry collision mesh filename=root/meshes/_1_________1__1__Body1_collision.stl; visual mesh filename=root/meshes/_1_________1__1__Body1.stl scale=1 1 1
- link 2сустав__1__1__body1: geometry collision mesh filename=root/meshes/_2________1__1__Body1_collision.stl; visual mesh filename=root/meshes/_2________1__1__Body1.stl scale=1 1 1
- link gripper_x_t__1__1__body21: geometry collision mesh filename=root/meshes/Component34_1__Body1_collision.stl; collision mesh filename=root/meshes/Component35_1__Body1_collision.stl
- link root: geometry collision mesh filename=root/meshes/Nema17__1___1___1__1__Body1_collision.stl; collision mesh filename=root/meshes/___________1___1___1__1__Body2_collision.stl
- link верхняя_крышка__1___1___1__1__body1: geometry collision mesh filename=root/meshes/________________1___1___1__1__Body1_collision.s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; visual mesh filename=root/meshes/________________1___1___1__1__Body1.stl scale=1 1 1
- link подставка__1___1___1__1__body1: geometry collision mesh filename=root/meshes/___________1___1___1__1__Body1_collision.stl; visual mesh filename=root/meshes/___________1___1___1__1__Body1.stl scale=1 1 1
- link ротор_основа__1___1___1__1__body1: geometry collision mesh filename=root/meshes/______________1___1___1__1__Body1_collision.stl; visual mesh filename=root/meshes/______________1___1___1__1__Body1.stl scale=1 1 1
- link соеденитель_захвата__1__1__body1: geometry collision mesh filename=root/meshes/_____________________1__1__Body1_collision.stl; visual mesh filename=root/meshes/_____________________1__1__Body1.stl scale=1 1 1
